File: hardware/SmartSwitch_V1_2.brd (EAGLE design)
At the start: 49 x 49 mm, 47 parts, among them K1 FTR-LYC5, K2 FTR-LYC5, U2 AMS1117-3.3

Commit message: Add files via upload
Parts:
- R7: value S14K275 -> S14K275GESPIEGELT; device varistor:S14K275 -> varistor:S14K275_
- flipped R7 to the top
Routing:
- net HV.N: track 49.5 -> 50.1 mm, vias 1 -> 0
Changed lines of the file:
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@@
 <layer number="23" name="tOrigins" color="15" fill="1" visible="yes" active="yes"/>
 <layer number="24" name="bOrigins" color="15" fill="1" visible="yes" active="yes"/>
-<layer number="25" name="tNames" color="7" fill="1" visible="yes" active="yes"/>
-<layer number="26" name="bNames" color="7" fill="1" visible="yes" active="yes"/>
-<layer number="27" name="tValues" color="7" fill="1" visible="yes" active="yes"/>
-<layer number="28" name="bValues" color="7" fill="1" visible="yes" active="yes"/>
+<layer number="25" name="tNames" color="7" fill="1" visible="no" active="yes"/>
+<layer number="26" name="bNames" color="7" fill="1" visible="no" active="yes"/>
+<layer number="27" name="tValues" color="7" fill="1" visible="no" active="yes"/>
+<layer number="28" name="bValues" color="7" fill="1" visible="no" active="yes"/>
 <layer number="29" name="tStop" color="7" fill="3" visible="no" active="yes"/>
 <layer number="30" name="bStop" color="7" fill="6" visible="no" active="yes"/>
@@
 <attribute name="VALUE" x="17.54" y="19.27" size="1.27" layer="28" rot="MR270"/>
 </element>
-<element name="R7" library="varistor" package="S14K275" value="S14K275" x="32" y="26.5" smashed="yes" rot="MR0">
-<attribute name="VALUE" x="35.429" y="26.119" size="1.27" layer="28" ratio="10" rot="MR90"/>
+<element name="R7" library="varistor" package="S14K275_" value="S14K275GESPIEGELT" x="32" y="26.5" smashed="yes">
+<attribute name="VALUE" x="28.571" y="26.119" size="1.27" layer="27" ratio="10" rot="R90"/>
 </element>
 <element name="F1" library="fuse" package="SMD_FUSE_HOLDER" value="0,4A" x="25" y="43.5" smashed="yes" rot="MR180"/>
@@
 <wire x1="17" y1="35.5" x2="26.5" y2="35.5" width="0.4064" layer="1"/>
 <wire x1="26.5" y1="35.5" x2="27.25" y2="34.75" width="0.4064" layer="1"/>
-<wire x1="27.25" y1="34.75" x2="27.25" y2="29.25" width="0.4064" layer="1"/>
-<wire x1="27.25" y1="29.25" x2="30.349" y2="26.151" width="0.4064" layer="1"/>
-<wire x1="30.349" y1="26.151" x2="33.651" y2="22.69" width="0.4064" layer="16"/>
+<wire x1="27.25" y1="34.75" x2="27.25" y2="28" width="0.4064" layer="1"/>
 <contactref element="R2" pad="1"/>
 <contactref element="R4" pad="1"/>
@@
 <wire x1="18.75" y1="46.25" x2="18.75" y2="40.25" width="0.4064" layer="16"/>
 <wire x1="18.75" y1="40.25" x2="17" y2="38.5" width="0.4064" layer="16"/>
-<via x="30.349" y="26.151" extent="1-16" drill="0.6" shape="octagon"/>
 <wire x1="12.422" y1="46" x2="14.25" y2="46" width="0.4064" layer="16"/>
 <wire x1="14.25" y1="46" x2="14.922" y2="46.672" width="0.4064" layer="16"/>
 <wire x1="14.922" y1="46.672" x2="17" y2="46.672" width="0.4064" layer="16"/>
+<wire x1="27.25" y1="28" x2="32.524" y2="22.726" width="0.4064" layer="1"/>
+<wire x1="32.524" y1="22.726" x2="33.524" y2="22.69" width="0.4064" layer="1"/>
 </signal>
 <signal name="N$8">
@@
 <wire x1="28.19" y1="43.31" x2="28" y2="43.5" width="1" layer="16"/>
 <wire x1="28.19" y1="43.46" x2="28.19" y2="43.31" width="1" layer="16"/>
-<wire x1="29.5" y1="34" x2="30.349" y2="33.151" width="0.4064" layer="16"/>
-<wire x1="30.349" y1="33.151" x2="30.349" y2="30.31" width="0.4064" layer="16"/>
+<wire x1="29.5" y1="34" x2="30.476" y2="33.024" width="0.4064" layer="16"/>
+<wire x1="30.476" y1="33.024" x2="30.476" y2="30.31" width="0.4064" layer="16"/>
 </signal>
 <signal name="RESET">

Commit message: Add files via upload
Parts:
- R7: value S14K275GESPIEGELT -> S14K275
- moved P 14.0 mm to (33.2, 43.2), flipped to the bottom
- moved KREUZ2 1.75 mm to (40.2, 42.2)
Routing:
- net I1.►: track 17.9 -> 29.6 mm, vias 0 -> 2
- net HV.P: track 36.2 -> 33.1 mm, vias 0 -> 2
- net O2.▼: track 9.29 -> 10.0 mm
- net N$5: track 24.8 -> 24.3 mm

Commit message: Add files via upload
Parts:
- R5, R6: value 47k -> 220k
Changed lines of the file:
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@@
 <grid distance="1" unitdist="mm" unit="mm" style="lines" multiple="1" display="yes" altdistance="0.125" altunitdist="mm" altunit="mm"/>
 <layers>
-<layer number="1" name="Top" color="17" fill="1" visible="yes" active="yes"/>
-<layer number="16" name="Bottom" color="16" fill="1" visible="yes" active="yes"/>
+<layer number="1" name="Top" color="17" fill="1" visible="no" active="yes"/>
+<layer number="16" name="Bottom" color="16" fill="1" visible="no" active="yes"/>
 <layer number="17" name="Pads" color="2" fill="1" visible="yes" active="yes"/>
-<layer number="18" name="Vias" color="2" fill="1" visible="yes" active="yes"/>
+<layer number="18" name="Vias" color="2" fill="1" visible="no" active="yes"/>
 <layer number="19" name="Unrouted" color="13" fill="1" visible="no" active="yes"/>
 <layer number="20" name="Dimension" color="15" fill="1" visible="yes" active="yes"/>
 <layer number="21" name="tPlace" color="7" fill="1" visible="yes" active="yes"/>
-<layer number="22" name="bPlace" color="7" fill="1" visible="yes" active="yes"/>
-<layer number="23" name="tOrigins" color="15" fill="1" visible="yes" active="yes"/>
-<layer number="24" name="bOrigins" color="15" fill="1" visible="yes" active="yes"/>
-<layer number="25" name="tNames" color="15" fill="1" visible="no" active="yes"/>
+<layer number="22" name="bPlace" color="7" fill="1" visible="no" active="yes"/>
+<layer number="23" name="tOrigins" color="15" fill="1" visible="no" active="yes"/>
+<layer number="24" name="bOrigins" color="15" fill="1" visible="no" active="yes"/>
+<layer number="25" name="tNames" color="15" fill="1" visible="yes" active="yes"/>
 <layer number="26" name="bNames" color="15" fill="1" visible="no" active="yes"/>
-<layer number="27" name="tValues" color="15" fill="1" visible="no" active="yes"/>
+<layer number="27" name="tValues" color="15" fill="1" visible="yes" active="yes"/>
 <layer number="28" name="bValues" color="15" fill="1" visible="no" active="yes"/>
-<layer number="29" name="tStop" color="17" fill="1" visible="no" active="yes"/>
+<layer number="29" name="tStop" color="17" fill="1" visible="yes" active="yes"/>
 <layer number="30" name="bStop" color="16" fill="1" visible="no" active="yes"/>
 <layer number="31" name="tCream" color="7" fill="4" visible="no" active="yes"/>
@@
 <layer number="49" name="Reference" color="7" fill="1" visible="no" active="yes"/>
 <layer number="50" name="dxf" color="7" fill="1" visible="no" active="no"/>
-<layer number="51" name="tDocu" color="7" fill="1" visible="no" active="yes"/>
+<layer number="51" name="tDocu" color="7" fill="1" visible="yes" active="yes"/>
 <layer number="52" name="bDocu" color="7" fill="1" visible="no" active="yes"/>
 <layer number="53" name="tGND_GNDA" color="7" fill="9" visible="no" active="no"/>
@@
 <layer number="131" name="tAdjust" color="7" fill="1" visible="no" active="no"/>
 <layer number="132" name="bAdjust" color="7" fill="1" visible="no" active="no"/>
-<layer number="133" name="bottom_silk" color="7" fill="1" visible="yes" active="yes"/>
+<layer number="133" name="bottom_silk" color="7" fill="1" visible="no" active="yes"/>
 <layer number="144" name="DrillLegend" color="7" fill="1" visible="no" active="no"/>
 <layer number="150" name="Notes" color="7" fill="1" visible="no" active="yes"/>
@@
 <attribute name="VALUE" x="18.79" y="45.52" size="0.6" layer="28" rot="MR270"/>
 </element>
-<element name="R5" library="rcl" package="R1206" value="47k" x="9.5" y="18.5" smashed="yes" rot="MR270">
+<element name="R5" library="rcl" package="R1206" value="220k" x="9.5" y="18.5" smashed="yes" rot="MR270">
 <attribute name="NAME" x="8.23" y="19.77" size="0.6" layer="26" rot="MR270"/>
 <attribute name="VALUE" x="8.165" y="18.02" size="0.6" layer="28" rot="MR270"/>
 </element>
-<element name="R6" library="rcl" package="R1206" value="47k" x="17.5" y="17" smashed="yes" rot="MR270">
+<element name="R6" library="rcl" package="R1206" value="220k" x="17.5" y="17" smashed="yes" rot="MR270">
 <attribute name="NAME" x="19.355" y="16.52" size="0.6" layer="26" rot="MR270"/>
 <attribute name="VALUE" x="19.29" y="18.645" size="0.6" layer="28" rot="MR270"/>
@@
 </element>
 <element name="UART" library="pinhead" package="1X03_SMALL" value="3" x="9" y="25.5" smashed="yes" rot="R180">
-<attribute name="NAME" x="6.4888" y="27.7962" size="1.27" layer="133" font="vector" ratio="12" rot="MR180"/>
+<attribute name="NAME" x="0.4888" y="26.1712" size="1.27" layer="133" font="vector" ratio="12" rot="MR180"/>
 </element>
 <element name="I²C" library="pinhead" package="1X04_SMALL" value="4" x="36" y="5.5" smashed="yes">
